Commit message: 6.2.6 添加虚拟部件,贴合地面

File: 666/ws/src/szcbot_description/urdf/szcbot/base.urdf.xacro (robot description, xacro)
@@ -2,4 +2,5 @@
 <robot xmlns:xacro="http://www.ros.org/wiki/xacro">
     <xacro:macro name="base_xacro" params="length radius">
+    <link name="base_footprint"/>
     <!-- 机器人的身体部分 -->
     <link name="base_link">
@@ -19,4 +20,12 @@
         </visual>
     </link>
+    <joint name="base_joint" type="fixed">
+        <!-- 关节的父部件 -->
+        <parent link="base_footprint"/>
+        <!-- 关节的子部件 -->
+        <child link="base_link"/>
+        <!-- 关节的偏移和旋转 -->
+        <origin xyz="0.0 0.0 ${length/2.0+0.032-0.001}" rpy="0.0 0.0 0.0"/>
+    </joint>
     </xacro:macro>
 </robot>
