Commit message: 6.3.1 添加碰撞属性

File: 666/ws/src/szcbot_description/urdf/szcbot/actuator/caster.urdf.xacro (robot description, xacro)
@@ -17,4 +17,16 @@
             </material>
         </visual>
+        <collision>
+        <!-- 沿着自己几何中心的偏移和旋转 -->
+            <origin xyz="0.0 0.0 0.0" rpy=" 0.0 0.0 0.0"/>
+            <!-- 几何形状 -->
+            <geometry>
+                <sphere radius="0.016"/>
+            </geometry>
+            <!-- 材质和颜色 -->
+            <material name="yellow">
+                <color rgba="1.0 1.0 0.0 0.85"/>
+            </material>
+        </collision>
     </link>
         <!-- 机器人的关节，用于组合各个部件 -->

File: 666/ws/src/szcbot_description/urdf/szcbot/actuator/whell.urdf.xacro (robot description, xacro)
@@ -17,4 +17,16 @@
             </material>
         </visual>
+        <collision>
+        <!-- 沿着自己几何中心的偏移和旋转 -->
+            <origin xyz="0.0 0.0 0.0" rpy="1.57079 0.0 0.0"/>
+            <!-- 几何形状 -->
+            <geometry>
+                <cylinder radius="0.0325" length="0.04"/>
+            </geometry>
+            <!-- 材质和颜色 -->
+            <material name="yellow">
+                <color rgba="1.0 1.0 0.0 0.85"/>
+            </material>
+        </collision>
     </link>
         <!-- 机器人的关节，用于组合各个部件 -->

File: 666/ws/src/szcbot_description/urdf/szcbot/base.urdf.xacro (robot description, xacro)
@@ -19,4 +19,17 @@
             </material>
         </visual>
+        <collision>
+        <!-- 沿着自己几何中心的偏移和旋转 -->
+            <origin xyz="0.0 0.0 0.0" rpy="0.0 0.0 0.0"/>
+            <!-- 几何形状 -->
+            <geometry>
+                <!-- 圆柱体 半径0.10m，高度0.12m -->
+                <cylinder radius="${radius}" length="${length}"/>
+            </geometry>
+            <!-- 材质和颜色 -->
+            <material name="white">
+                <color rgba="1.0 1.0 1.0 0.5"/>
+            </material>
+        </collision>
     </link>
     <joint name="base_joint" type="fixed">

File: 666/ws/src/szcbot_description/urdf/szcbot/sensor/camera.urdf.xacro (robot description, xacro)
@@ -17,4 +17,16 @@
             </material>
         </visual>
+        <collision>
+        <!-- 沿着自己几何中心的偏移和旋转 -->
+            <origin xyz="0.0 0.0 0.0" rpy="0.0 0.0 0.0"/>
+            <!-- 几何形状 -->
+            <geometry>
+                <box size="0.02 0.10 0.02"/>
+            </geometry>
+            <!-- 材质和颜色 -->
+            <material name="black">
+                <color rgba="0.0 0.0 0.0 0.5"/>
+            </material>
+        </collision>
     </link>
         <!-- 机器人的关节，用于组合各个部件 -->

File: 666/ws/src/szcbot_description/urdf/szcbot/sensor/imu.urdf.xacro (robot description, xacro)
@@ -18,4 +18,17 @@
             </material>
         </visual>
+        <collision>
+        <!-- 沿着自己几何中心的偏移和旋转 -->
+            <origin xyz="0.0 0.0 0.0" rpy="0.0 0.0 0.0"/>
+            <!-- 几何形状 -->
+            <geometry>
+                <!-- 正方体0.02m x 0.02m x 0.02m -->
+                <box size="0.02 0.02 0.02"/>
+            </geometry>
+            <!-- 材质和颜色 -->
+            <material name="black">
+                <color rgba="0.0 0.0 0.0 0.5"/>
+            </material>
+        </collision>
     </link>
         <!-- 机器人的关节，用于组合各个部件 -->

File: 666/ws/src/szcbot_description/urdf/szcbot/sensor/laser.urdf.xacro (robot description, xacro)
@@ -17,4 +17,16 @@
             </material>
         </visual>
+        <collision>
+                <!-- 沿着自己几何中心的偏移和旋转 -->
+            <origin xyz="0.0 0.0 0.0" rpy="0.0 0.0 0.0"/>
+            <!-- 几何形状 -->
+            <geometry>
+                <cylinder radius="0.01" length="0.10"/>
+            </geometry>
+            <!-- 材质和颜色 -->
+            <material name="black">
+                <color rgba="0.0 0.0 0.0 1.0"/>
+            </material>
+        </collision>
     </link>
     <!-- 激光雷达的主体 -->
@@ -32,4 +44,16 @@
             </material>
         </visual>
+         <collision>
+                 <!-- 沿着自己几何中心的偏移和旋转 -->
+            <origin xyz="0.0 0.0 0.0" rpy="0.0 0.0 0.0"/>
+            <!-- 几何形状 -->
+            <geometry>
+                <cylinder radius="0.02" length="0.02"/>
+            </geometry>
+            <!-- 材质和颜色 -->
+            <material name="black">
+                <color rgba="0.0 0.0 0.0 1.0"/>
+            </material>
+        </collision>
     </link>
         <!-- 机器人的关节，用于组合各个部件 -->

Commit message: 6.4.3 使用Gazebo标签扩展URDF

File: 666/ws/src/szcbot_description/urdf/szcbot/actuator/caster.urdf.xacro (robot description, xacro)
@@ -41,4 +41,11 @@
         <origin xyz="${xyz}" rpy="0.0 0.0 0.0"/>
     </joint>
+                    <gazebo reference ="${caster_name}_link">
+        <material>Gazebo/Yellow</material>
+        <mu1 value="0.0"/>
+        <mu2 value="0.0"/>
+        <kp value="1000000000.0"/>
+        <kd value="1.0"/>
+    </gazebo>
     </xacro:macro>
 </robot>

File: 666/ws/src/szcbot_description/urdf/szcbot/actuator/whell.urdf.xacro (robot description, xacro)
@@ -42,4 +42,11 @@
         <axis xyz="0.0 1.0 0.0"/>
     </joint>
+                <gazebo reference ="${wheel_name}_link">
+        <material>Gazebo/Yellow</material>
+        <mu1 value="20.0"/>
+        <mu2 value="20.0"/>
+        <kp value="1000000000.0"/>
+        <kd value="1.0"/>
+    </gazebo>
     </xacro:macro>
 </robot>

File: 666/ws/src/szcbot_description/urdf/szcbot/base.urdf.xacro (robot description, xacro)
@@ -44,4 +44,7 @@
         <origin xyz="0.0 0.0 ${length/2.0+0.032-0.001}" rpy="0.0 0.0 0.0"/>
     </joint>
+        <gazebo reference ="base_link">
+        <material>Gazebo/Blue</material>
+    </gazebo>
     </xacro:macro>
 </robot>

File: 666/ws/src/szcbot_description/urdf/szcbot/sensor/camera.urdf.xacro (robot description, xacro)
@@ -41,4 +41,7 @@
         <origin xyz="${xyz}" rpy="0.0 0.0 0.0"/>
     </joint>
+            <gazebo reference ="camera_link">
+        <material>Gazebo/Black</material>
+    </gazebo>
     </xacro:macro>
 </robot>

File: 666/ws/src/szcbot_description/urdf/szcbot/sensor/imu.urdf.xacro (robot description, xacro)
@@ -43,4 +43,7 @@
         <origin xyz="${xyz}" rpy="0.0 0.0 0.0"/>
     </joint>
+        <gazebo reference ="imu_link">
+        <material>Gazebo/Red</material>
+    </gazebo>
     </xacro:macro>
 </robot>

File: 666/ws/src/szcbot_description/urdf/szcbot/sensor/laser.urdf.xacro (robot description, xacro)
@@ -77,4 +77,11 @@
         <origin xyz="${xyz}" rpy="0.0 0.0 0.0"/>
     </joint>
+    <!-- gazebo标签-->
+    <gazebo reference ="laser_cylinder_link">
+        <material>Gazebo/Black</material>
+    </gazebo>
+    <gazebo reference ="laser_link">
+        <material>Gazebo/Black</material>
+    </gazebo>
     </xacro:macro>
 </robot>

File: 666/ws/src/szcbot_description/urdf/szcbot/szcbot.urdf.xacro (robot description, xacro)
@@ -12,5 +12,5 @@
 <xacro:base_xacro length="0.12" radius="0.10"/>
 <xacro:imu_xacro xyz="0.0 0.0 0.02"/>
-<xacro:camera_xacro xyz="0.10 0.0 0.075"/>
+<xacro:camera_xacro xyz="0.10 0.0 0.07"/>
 <xacro:laser_xacro  xyz="0.00 0.0 0.11"/>
 <xacro:wheel_xacro wheel_name="left_wheel" xyz="0.0 0.10 -0.06"/>
