Commit message: 7.2.2 将地图保存为文件

File: 777/ws/src/szcbot_description/urdf/first_robot.xacro (robot description, xacro)
@@ -1,7 +1,5 @@
 <?xml version="1.0"?>
-<robot xmlns:xacro="http://www.ros.org/wiki/xacro">
-    <xacro:include filename="$(find szcbot_description)/urdf/szcbot/common_inertia.xacro"/>
-    <xacro:macro name="base_xacro" params="length radius">
-    <link name="base_footprint"/>
+<robot xmlns:xacro="http://www.ros.org/wiki/xacro" name="first_robot">
+    <xacro:macro name="base_link" params="length radius">
     <!-- 机器人的身体部分 -->
     <link name="base_link">
@@ -20,31 +18,36 @@
             </material>
         </visual>
-        <collision>
+    </link>
+    </xacro:macro>
+    <!-- 机器人的IMU部件，惯性测量传感器 -->
+        <xacro:macro name="imu_link" params="imu_name xyz">
+        <link name="${imu_name}_link">
+        <!-- 部件的外观描述 -->
+        <visual>
         <!-- 沿着自己几何中心的偏移和旋转 -->
             <origin xyz="0.0 0.0 0.0" rpy="0.0 0.0 0.0"/>
             <!-- 几何形状 -->
             <geometry>
-                <!-- 圆柱体 半径0.10m，高度0.12m -->
-                <cylinder radius="${radius}" length="${length}"/>
+                <!-- 正方体0.02m x 0.02m x 0.02m -->
+                <box size="0.02 0.02 0.02"/>
             </geometry>
             <!-- 材质和颜色 -->
-            <material name="white">
-                <color rgba="1.0 1.0 1.0 0.5"/>
+            <material name="black">
+                <color rgba="0.0 0.0 0.0 0.5"/>
             </material>
-        </collision>
-        <!-- 机器人的惯性描述 -->
-        <xacro:cylinder_inertia m="2.0" r="${radius}" h="${length}" />
+        </visual>
     </link>
-    <joint name="base_joint" type="fixed">
+        <!-- 机器人的关节，用于组合各个部件 -->
+    <joint name="${imu_name}_joint" type="fixed">
         <!-- 关节的父部件 -->
-        <parent link="base_footprint"/>
+        <parent link="base_link"/>
         <!-- 关节的子部件 -->
-        <child link="base_link"/>
+        <child link="${imu_name}_link"/>
         <!-- 关节的偏移和旋转 -->
-        <origin xyz="0.0 0.0 ${length/2.0+0.032-0.001}" rpy="0.0 0.0 0.0"/>
+        <origin xyz="${xyz}" rpy="0.0 0.0 0.0"/>
     </joint>
-        <gazebo reference ="base_link">
-        <material>Gazebo/Blue</material>
-    </gazebo>
     </xacro:macro>
+<xacro:base_link length="0.12" radius="0.10"/>
+<xacro:imu_link imu_name="imu" xyz="0.0 0.0 0.06"/>
+<xacro:imu_link imu_name="imu_down" xyz="0.0 0.0 -0.06"/>
 </robot>

File: 777/ws/src/szcbot_description/urdf/szcbot/base.urdf.xacro (robot description, xacro)
@@ -34,5 +34,5 @@
         </collision>
         <!-- 机器人的惯性描述 -->
-        <xacro:cylinder_inertia m="2.0" r="${radius}" h="${length}" />
+        <xacro:cylinder_inertia m="1.0" r="${radius}" h="${length}" />
     </link>
     <joint name="base_joint" type="fixed">

File: 777/ws/src/szcbot_description/urdf/szcbot/plugins/gazebo_sensor_plugin.xacro (robot description, xacro)
@@ -9,6 +9,6 @@
                 <!-- 发布话题名称 -->
                 <topic>lidar</topic>
-                <!-- 更新频率 100Hz -->
-                <update_rate>100</update_rate>
+                <!-- 更新频率 10Hz -->
+                <update_rate>10</update_rate>
                 <lidar>
                     <!-- 设置扫描范围 -->

File: 777/ws/src/szcbot_description/urdf/szcbot/sensor/imu.urdf.xacro (robot description, xacro)
@@ -2,8 +2,7 @@
 <robot xmlns:xacro="http://www.ros.org/wiki/xacro">
     <xacro:include filename="$(find szcbot_description)/urdf/szcbot/common_inertia.xacro"/>
-    <xacro:macro name="base_xacro" params="length radius">
-    <link name="base_footprint"/>
-    <!-- 机器人的身体部分 -->
-    <link name="base_link">
+    <!-- 机器人的IMU部件，惯性测量传感器 -->
+        <xacro:macro name="imu_xacro" params="xyz">
+        <link name="imu_link">
         <!-- 部件的外观描述 -->
         <visual>
@@ -12,10 +11,10 @@
             <!-- 几何形状 -->
             <geometry>
-                <!-- 圆柱体 半径0.10m，高度0.12m -->
-                <cylinder radius="${radius}" length="${length}"/>
+                <!-- 正方体0.02m x 0.02m x 0.02m -->
+                <box size="0.02 0.02 0.02"/>
             </geometry>
             <!-- 材质和颜色 -->
-            <material name="white">
-                <color rgba="1.0 1.0 1.0 0.5"/>
+            <material name="black">
+                <color rgba="0.0 0.0 0.0 0.5"/>
             </material>
         </visual>
@@ -25,25 +24,25 @@
             <!-- 几何形状 -->
             <geometry>
-                <!-- 圆柱体 半径0.10m，高度0.12m -->
-                <cylinder radius="${radius}" length="${length}"/>
+                <!-- 正方体0.02m x 0.02m x 0.02m -->
+                <box size="0.02 0.02 0.02"/>
             </geometry>
             <!-- 材质和颜色 -->
-            <material name="white">
-                <color rgba="1.0 1.0 1.0 0.5"/>
+            <material name="black">
+                <color rgba="0.0 0.0 0.0 0.5"/>
             </material>
         </collision>
-        <!-- 机器人的惯性描述 -->
-        <xacro:cylinder_inertia m="2.0" r="${radius}" h="${length}" />
+        <xacro:box_inertia m="0.05" w="0.02" h="0.02" d="0.02" />
     </link>
-    <joint name="base_joint" type="fixed">
+        <!-- 机器人的关节，用于组合各个部件 -->
+    <joint name="imu_joint" type="fixed">
         <!-- 关节的父部件 -->
-        <parent link="base_footprint"/>
+        <parent link="base_link"/>
         <!-- 关节的子部件 -->
-        <child link="base_link"/>
+        <child link="imu_link"/>
         <!-- 关节的偏移和旋转 -->
-        <origin xyz="0.0 0.0 ${length/2.0+0.032-0.001}" rpy="0.0 0.0 0.0"/>
+        <origin xyz="${xyz}" rpy="0.0 0.0 0.0"/>
     </joint>
-        <gazebo reference ="base_link">
-        <material>Gazebo/Blue</material>
+        <gazebo reference ="imu_link">
+        <material>Gazebo/Red</material>
     </gazebo>
     </xacro:macro>

File: 777/ws/src/szcbot_description/urdf/szcbot/szcbot.urdf.xacro (robot description, xacro)
@@ -18,6 +18,6 @@
 <xacro:camera_xacro xyz="0.10 0.0 0.07"/>
 <xacro:laser_xacro  xyz="0.00 0.0 0.11"/>
-<xacro:wheel_xacro wheel_name="left_wheel" xyz="0.0 0.10 -0.0585"/>
-<xacro:wheel_xacro wheel_name="right_wheel" xyz="0.0 -0.10 -0.0585"/>
+<xacro:wheel_xacro wheel_name="left_wheel" xyz="0.0 0.10 -0.06"/>
+<xacro:wheel_xacro wheel_name="right_wheel" xyz="0.0 -0.10 -0.06"/>
 <xacro:caster_xacro caster_name="front_caster" xyz="0.08 0.0 -0.076"/>
 <xacro:caster_xacro caster_name="back_caster" xyz="-0.08 0.0 -0.076"/>
